File: hardware/kicad/opensolder.kicad_pcb (KiCad board)
At the start: 2 copper layers, 100 x 44 mm, 69 parts, among them J1 AC_Input, J2 Hirose RPC1-12RB-6P(71), J3 SWD, J4 UART, J5 Reset_Switch, Q1 KIA50N06BD, Q2 KIA50N06BD, SW2 PEC11R-RotEnc, U1 VOS628A, U2 L78L24_SOT89, U3 Si8751, U4 AP2111H-3.3, U5 MAX4238ASA, U6 OLED, U7 STM32F072CBTx, U8 PCT2075GV, Y1 Crystal_8MHz

Commit message: Schematic update.
Parts:
- removed C18: 100n, Capacitor_SMD:C_0805_2012Metric
- removed C6: 1u, Capacitor_SMD:C_1210_3225Metric
- removed F1: Fast 12A, Fuse:Fuseholder_Cylinder-5x20mm_Schurter_0031_8201_Horizontal_Open
- removed PS1: PDSE1-S24-S5-S, 0_Howie:PDSE1_DCDC
- removed R18: 100k, Resistor_SMD:R_0805_2012Metric
- removed R20: 3k3, Resistor_SMD:R_0805_2012Metric
- removed TP1: ZeroCross, TestPoint:TestPoint_Pad_D1.0mm
- removed TP2: +24V, TestPoint:TestPoint_Pad_D1.0mm
- removed TP3: Heater, TestPoint:TestPoint_Pad_D1.0mm
- removed TP4: +5V, TestPoint:TestPoint_Pad_D1.0mm
- removed U3: Si8751, Package_SO:SOIC-8_3.9x4.9mm_P1.27mm
- removed U7: STM32F072CBTx, Package_QFP:LQFP-48_7x7mm_P0.5mm
- removed U8: PCT2075GV, Package_SO:TSOP-6_1.65x3.05mm_P0.95mm
- removed Y1: Crystal_8MHz, Crystal:Crystal_SMD_HC49-SD
- added C22: 220p, Capacitor_SMD:C_0603_1608Metric_Pad1.08x0.95mm_HandSolder, F.Cu at (213.7, 101.7)
- added C32: 100u, Capacitor_THT:CP_Radial_D8.0mm_P3.50mm, F.Cu at (226.3, 93.7)
- added C45: 100n, Capacitor_SMD:C_0603_1608Metric_Pad1.08x0.95mm_HandSolder, F.Cu at (213.7, 104.2)
- added D11: 1N4148WS, Diode_SMD:D_SOD-323, F.Cu at (218.1, 106.6)
- added J6: Conn_01x04_Pin, Connector_PinHeader_2.54mm:PinHeader_1x04_P2.54mm_Vertical, F.Cu at (227.1, 102.7)
- added Q3: IRF9540N, Package_TO_SOT_THT:TO-220-3_Vertical, F.Cu at (214.8, 82.8)
- added Q4: IRF9540N, Package_TO_SOT_THT:TO-220-3_Vertical, F.Cu at (214.8, 88.7)
- added Q5: IRF9540N, Package_TO_SOT_THT:TO-220-3_Vertical, F.Cu at (214.8, 94.7)
- added Q6: MMBT5551L, Package_TO_SOT_SMD:SOT-23, F.Cu at (229.9, 81.2)
- added Q7: MMBT5551L, Package_TO_SOT_SMD:SOT-23, F.Cu at (229.9, 85.9)
- added R21: 1k, Resistor_SMD:R_0603_1608Metric_Pad0.98x0.95mm_HandSolder, F.Cu at (225.3, 80.1)
- added R22: 10k, Resistor_SMD:R_0603_1608Metric_Pad0.98x0.95mm_HandSolder, F.Cu at (225.3, 82.6)
- added R23: 10k, Resistor_SMD:R_0603_1608Metric_Pad0.98x0.95mm_HandSolder, F.Cu at (225.3, 85.1)
- added R24: 22k, Resistor_SMD:R_0603_1608Metric_Pad0.98x0.95mm_HandSolder, F.Cu at (213.7, 106.7)
- added R25: 1k, Resistor_SMD:R_0603_1608Metric_Pad0.98x0.95mm_HandSolder, F.Cu at (213.7, 109.2)
- added R27: 22k, Resistor_SMD:R_0603_1608Metric_Pad0.98x0.95mm_HandSolder, F.Cu at (213.7, 111.7)
- added R55: 1k, Resistor_SMD:R_0603_1608Metric_Pad0.98x0.95mm_HandSolder, F.Cu at (225.3, 87.6)
- added U17: Screen, opensolder:WC1602A, B.Cu at (182.0, 57.5)
- added U9: NCS21802DMR2G, Package_SO:OnSemi_Micro8, F.Cu at (219.3, 102.8)
- C1: value 47u -> 10n; footprint Capacitor_THT:CP_Radial_D8.0mm_P3.50mm -> Capacitor_SMD:C_0603_1608Metric_Pad1.08x0.95mm_HandSolder
- C10: value 20p -> 10n; footprint Capacitor_SMD:C_0805_2012Metric -> Capacitor_SMD:C_0603_1608Metric_Pad1.08x0.95mm_HandSolder
- C11, C2, C3: value 1u -> 100n; footprint Capacitor_SMD:C_1210_3225Metric -> Capacitor_SMD:C_0603_1608Metric_Pad1.08x0.95mm_HandSolder
- C12, C13, C19, C7, C8: footprint Capacitor_SMD:C_0805_2012Metric -> Capacitor_SMD:C_0603_1608Metric_Pad1.08x0.95mm_HandSolder
- C14, C15, C16: value 100n -> 10n; footprint Capacitor_SMD:C_0805_2012Metric -> Capacitor_SMD:C_0603_1608Metric_Pad1.08x0.95mm_HandSolder
- C17: value 100n -> 1u; footprint Capacitor_SMD:C_0805_2012Metric -> Capacitor_SMD:C_0603_1608Metric_Pad1.08x0.95mm_HandSolder
- C20: value 10n -> 10u; footprint Capacitor_SMD:C_0805_2012Metric -> Capacitor_SMD:C_0603_1608Metric_Pad1.08x0.95mm_HandSolder
- C21: value 10n -> 1u; footprint Capacitor_SMD:C_0805_2012Metric -> Capacitor_SMD:C_0603_1608Metric_Pad1.08x0.95mm_HandSolder
- C4: value 1u -> 10u; footprint Capacitor_SMD:C_1210_3225Metric -> Capacitor_SMD:C_0603_1608Metric_Pad1.08x0.95mm_HandSolder
- C5: value 100n -> 100u; footprint Capacitor_SMD:C_0805_2012Metric -> Capacitor_THT:CP_Radial_D8.0mm_P3.50mm
- C9: value 20p -> 100n; footprint Capacitor_SMD:C_0805_2012Metric -> Capacitor_SMD:C_0603_1608Metric_Pad1.08x0.95mm_HandSolder
- D1: value MB6S-TP -> 1N4148WS; footprint Package_TO_SOT_SMD:TO-269AA -> Diode_SMD:D_SOD-323
- D2, D3: value S1M -> 1N4148WS; footprint Diode_SMD:D_SMA -> Diode_SMD:D_SOD-323
- J1: value AC_Input -> DC_Input
- J5: value Reset_Switch -> RESET
- Q1: value KIA50N06BD -> MMBT5401; footprint Package_TO_SOT_SMD:TO-252-2 -> Package_TO_SOT_SMD:SOT-23
- Q2: value KIA50N06BD -> MMBT5551L; footprint Package_TO_SOT_SMD:TO-252-2 -> Package_TO_SOT_SMD:SOT-23
- R1, R10, R11, R12, R13, R14, R15, R16, R17, R2, R3, R7, R9: footprint Resistor_SMD:R_0805_2012Metric -> Resistor_SMD:R_0603_1608Metric_Pad0.98x0.95mm_HandSolder
- R19: value 3k3 -> 100k; footprint Resistor_SMD:R_0805_2012Metric -> Resistor_SMD:R_0603_1608Metric_Pad0.98x0.95mm_HandSolder
- R4: value 10k -> 22k; footprint Resistor_SMD:R_0805_2012Metric -> Resistor_SMD:R_0603_1608Metric_Pad0.98x0.95mm_HandSolder
- R5: value 10k -> 10 mOhm; footprint Resistor_SMD:R_0805_2012Metric -> Resistor_SMD:R_2512_6332Metric_Pad1.40x3.35mm_HandSolder
- R6: value 22k -> 100; footprint Resistor_SMD:R_0805_2012Metric -> Resistor_SMD:R_0603_1608Metric_Pad0.98x0.95mm_HandSolder
- R8: value 390 -> 10k; footprint Resistor_SMD:R_0805_2012Metric -> Resistor_SMD:R_0603_1608Metric_Pad0.98x0.95mm_HandSolder
- SW2: value PEC11R-RotEnc -> PEC11R-4220F-S0024
- U1: value VOS628A -> L7805; footprint Package_SO:SOP-4_4.4x2.6mm_P1.27mm -> Package_TO_SOT_THT:TO-220-3_Vertical
- U2: value L78L24_SOT89 -> LMT84LPM; footprint Package_TO_SOT_SMD:SOT-89-3 -> Package_TO_SOT_THT:TO-92_Inline_W4.0mm_Horizontal_FlatSideDown
- U5: value MAX4238ASA -> BluePill; footprint Package_SO:SOIC-8_3.9x4.9mm_P1.27mm -> opensolder:BluePill; moved to B.Cu
- moved U5 37.8 mm to (155.1, 80.6)
- moved C1 27.5 mm to (162.3, 120.5)
- moved C10 27.5 mm to (133.5, 134.5)
- moved C11 27.5 mm to (146.5, 132.5)
- moved C12 27.5 mm to (135.5, 120.5)
- moved C13 27.5 mm to (124.5, 120.5)
- moved C14 27.5 mm to (124.5, 130.5)
- moved C15 27.5 mm to (135.5, 130.5)
- moved C16 27.5 mm to (113.5, 145.0)
- moved C17 27.5 mm to (119.5, 143.0)
- moved C19 27.5 mm to (113.5, 142.5)
- moved C2 27.5 mm to (160.0, 132.5)
- moved C20 27.5 mm to (113.5, 137.5)
- moved C21 27.5 mm to (113.5, 140.0)
- moved C3 27.5 mm to (158.0, 138.0)
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Connections:
- C1 pad 1: Net-(C1-Pad1) -> GND
- C1 pad 2: Net-(C1-Pad2) -> THERMOCOUPLE+
- C10 pad 1: Net-(C10-Pad1) -> GND
- C10 pad 2: GND -> /MCU/ENC_A
- C11 pad 1: +3V3 -> GND
- C11 pad 2: GND -> +3V3
- C12 pad 1: +3V3 -> GND
- C12 pad 2: GND -> +3V3
- C13 pad 1: +3V3 -> GND
- C13 pad 2: GND -> +3V3
- C14 pad 1: +3V3 -> GND
- C14 pad 2: GND -> +3V3
- C15 pad 1: +3V3 -> GND
- C15 pad 2: GND -> +3V3
- C16 pad 1: /MCU/TIP_REMOVER -> GND
- C16 pad 2: GND -> /MCU/ENC_B
- C19 pad 1: /MCU/ENC_SW -> GND
- C19 pad 2: GND -> +3V3
- C2 pad 1: Net-(C2-Pad1) -> GND
- C2 pad 2: Net-(C1-Pad2) -> +3V3
- C20 pad 1: /MCU/ENC_A -> +24V
- C21 pad 1: /MCU/ENC_B -> +3V3
- C3 pad 1: +3V3 -> GND
- C3 pad 2: GND -> /MCU/TIP_REMOVER
- C5 pad 1: +3V3 -> +24V
- C5 pad 2: GND -> 0
- C7 pad 1: TIP_CLAMP -> THERMOCOUPLE-
- C7 pad 2: GND -> THERMOCOUPLE_ADC
- C8 pad 1: +3V3 -> GND
- C8 pad 2: GND -> /MCU/STAND
- C9 pad 1: /MCU/HSE_IN -> GND
- C9 pad 2: GND -> /MCU/ENC_SW
- D1 pad 1: Net-(D1-Pad1) -> THERMOCOUPLE-
- D1 pad 2: /AC/AC2 -> GND
- D2 pad 1: TIP_THERMOCOUPLE -> GND
- D2 pad 2: GND -> THERMOCOUPLE+
- D3 pad 2: TIP_THERMOCOUPLE -> THERMOCOUPLE-
- J1 pad 1: /AC/AC1 -> +24V
- J1 pad 2: GND -> unconnected-(J1-Pin_2-Pad2)
- J1 pad 3: /AC/AC2 -> GND
- J2 pad 1: GND -> Net-(J2-Pad1)
- J2 pad 2: TIP_THERMOCOUPLE -> SHUNT
- J2 pad 5: /AC/AC2 -> Net-(Q3-D)
- J5 pad 1: /MCU/NRST -> Net-(J5-Pin_1)
- Q1 pad 1: /AC/MOS_Gate -> Net-(Q1-B)
- Q1 pad 2: Net-(D1-Pad1) -> +24V
- Q1 pad 3: /AC/MOS_Source -> GATE
- Q2 pad 1: /AC/MOS_Gate -> Net-(Q2-B)
- Q2 pad 2: TIP_THERMOCOUPLE -> Net-(Q2-E)
- Q2 pad 3: /AC/MOS_Source -> GATE
- R1 pad 1: /AC/AC2 -> GATE
- R1 pad 2: Net-(R1-Pad2) -> Net-(Q2-B)
- R10 pad 1: /MCU/TIP_REMOVER_CONN -> Net-(R10-Pad1)
- R10 pad 2: /MCU/TIP_REMOVER -> /MCU/ENC_A
- R12 pad 1: /MCU/STAND_CONN -> Net-(R12-Pad1)
- R12 pad 2: /MCU/STAND -> /MCU/ENC_SW
- R13 pad 2: Net-(R13-Pad2) -> Net-(R12-Pad1)
- R14 pad 1: Net-(R13-Pad2) -> /MCU/STAND_CONN
- R14 pad 2: /MCU/ENC_SW -> /MCU/STAND
- R15 pad 2: Net-(R15-Pad2) -> Net-(R10-Pad1)
- R16 pad 1: Net-(R15-Pad2) -> /MCU/TIP_REMOVER_CONN
- R16 pad 2: /MCU/ENC_A -> /MCU/TIP_REMOVER
- R19 pad 1: +3V3 -> Net-(R17-Pad2)
- R19 pad 2: /MCU/SDA -> /MCU/ENC_B
- R2 pad 1: /AC/AC2 -> Net-(Q6-B)
- R2 pad 2: Net-(R1-Pad2) -> Net-(Q7-C)
- R3 pad 1: /AC/AC2 -> Net-(Q1-B)
- R3 pad 2: Net-(R1-Pad2) -> Net-(Q7-C)
- R4 pad 1: TIP_THERMOCOUPLE -> Net-(U9B--)
- R4 pad 2: TIP_CHECK -> SHUNT_ADC
- R5 pad 1: TIP_CLAMP -> SHUNT
- R5 pad 2: TIP_THERMOCOUPLE -> GND
- R6 pad 1: THERMOCOUPLE_ADC -> THERMOCOUPLE-
- R6 pad 2: Net-(R6-Pad2) -> Net-(J2-Pad1)
- R7 pad 1: Net-(R6-Pad2) -> THERMOCOUPLE+
- R7 pad 2: GND -> SHUNT
- R8 pad 1: Net-(C10-Pad1) -> +24V
- R8 pad 2: /MCU/HSE_OUT -> GATE
- SW2 pad A: Net-(R15-Pad2) -> Net-(R10-Pad1)
- SW2 pad S1: Net-(R13-Pad2) -> Net-(R12-Pad1)
- U1 pad 1: Net-(R1-Pad2) -> +24V
- U1 pad 2: Net-(D1-Pad1) -> GND
- U1 pad 3: GND -> +5V
- U2 pad 1: Net-(C2-Pad1) -> +3V3
- U2 pad 2: Net-(C1-Pad2) -> SW_TEMP
- U2 pad 3: Net-(C1-Pad1) -> GND_C
- U5 pad 1: +3V3 -> unconnected-(U5-PB12-Pad1)
- U5 pad 2: Net-(R6-Pad2) -> unconnected-(U5-PB13-Pad2)
- U5 pad 3: TIP_CLAMP -> unconnected-(U5-PB14-Pad3)
- U5 pad 4: GND -> unconnected-(U5-PB15-Pad4)
- U5 pad 6: THERMOCOUPLE_ADC -> /MCU/UART_TX
- U5 pad 7: +3V3 -> /MCU/UART_RX
Routing:
- net +3V3: track 209.6 -> 0.00 mm, vias 0 -> 6
- net TIP_THERMOCOUPLE: track 78.6 -> 0.00 mm
- net GND: track 51.5 -> 0.00 mm, vias 260 -> 255
- net /MCU/TIP_REMOVER_CONN: track 41.2 -> 0.00 mm
- net /MCU/STAND_CONN: track 40.6 -> 0.00 mm
- net TIP_CLAMP: track 40.1 -> 0.00 mm
- net ZERO_CROSS: track 38.8 -> 0.00 mm, vias 4 -> 0
- net HEATER: track 38.5 -> 0.00 mm
- net Net-(C2-Pad1): track 36.9 -> 0.00 mm
- net /MCU/STAND: track 32.3 -> 0.00 mm, vias 0 -> 1
- net /AC/AC2: track 31.1 -> 0.00 mm
- net /MCU/TIP_REMOVER: track 30.5 -> 0.00 mm
- net Net-(C1-Pad2): track 28.9 -> 0.00 mm
- net /MCU/ENC_SW: track 28.6 -> 0.00 mm
- net TIP_CHECK: track 28.6 -> 0.00 mm
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- added copper zone on F.Cu, net +24V
- added copper zone on B.Cu, net GATE
- added copper zone on F.Cu, net GATE
- added copper zone on F.Cu, net Net-(Q3-D)
- added copper zone on F.Cu, net SHUNT
- removed copper zone on F.Cu, net /AC/AC1
- removed copper zone on F.Cu, net /AC/AC2
- removed copper zone on B.Cu, net /AC/MOS_Source
- removed copper zone on F.Cu, net /AC/MOS_Source
- removed copper zone on F.Cu, net Net-(D1-Pad1)
- removed copper zone on F.Cu, net TIP_THERMOCOUPLE
Other:
- board size 100 x 44 mm -> 100 x 100 mm

Commit message: Placement???
Parts:
- removed C11, C12, C13: 100n, Capacitor_SMD:C_0603_1608Metric_Pad1.08x0.95mm_HandSolder
- removed C14, C15: 10n, Capacitor_SMD:C_0603_1608Metric_Pad1.08x0.95mm_HandSolder
- removed J1: DC_Input, Connector_Phoenix_MSTB:PhoenixContact_MSTBVA_2,5_3-G_1x03_P5.00mm_Vertical
- removed Q4, Q5: IRF9540N, Package_TO_SOT_THT:TO-220-3_Vertical
- removed U6: OLED, 0_Howie:OLED_SSD1306_SPI_1.54
- added C6: 1n, Capacitor_SMD:C_0603_1608Metric_Pad1.08x0.95mm_HandSolder, F.Cu at (166.0, 142.1)
- added J7: Screw_Terminal_01x02, TerminalBlock_Phoenix:TerminalBlock_Phoenix_MKDS-1,5-2-5.08_1x02_P5.08mm_Horizontal, F.Cu at (183.4, 109.0)
- C1: value 10n -> 1n
- C7: value 10n -> 1u
- Q3: value IRF9540N -> IRF5305
- moved C5 107.9 mm to (74.3, 206.2)
- moved J6 98.7 mm to (128.6, 109.1), turned to 90 degrees
- moved Q6 75.5 mm to (162.8, 115.9), turned to -90 degrees
- moved Q7 74.3 mm to (160.3, 111.9), turned to 90 degrees
- moved R23 72.7 mm to (159.3, 115.8), turned to -90 degrees
- moved D11 69.4 mm to (160.7, 145.6), turned to -90 degrees
- moved R21 66.2 mm to (166.2, 110.0)
- moved R55 66.1 mm to (165.6, 115.9), turned to 90 degrees
- moved R22 64.4 mm to (166.2, 108.4), turned to 180 degrees
- moved U9 63.1 mm to (171.1, 143.4)
- moved R24 62.8 mm to (164.4, 145.6), turned to -90 degrees
- moved TP5 61.0 mm to (113.8, 187.0)
- moved U17 58.7 mm to (190.4, 115.6)
- moved R27 57.9 mm to (164.4, 142.1), turned to -90 degrees
- moved C45 56.2 mm to (171.1, 140.8)
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Connections:
- C7 pad 1: THERMOCOUPLE- -> +3V3
- C7 pad 2: THERMOCOUPLE_ADC -> GND
- Q3 pad 3: Net-(Q3-S) -> +24V
Routing:
- net SHUNT: vias 1 -> 0
- net HEATER: vias 4 -> 0
- net GND: vias 255 -> 0
- net GATE: vias 8 -> 0
- net /MCU/TIP_REMOVER_CONN: vias 2 -> 0
- net /MCU/SWCLK: vias 2 -> 0
- net /MCU/STAND_CONN: vias 2 -> 0
- net /MCU/STAND: vias 1 -> 0
- net /MCU/ENC_B: vias 1 -> 0
- net +3V3: vias 6 -> 0
- net (no net): vias 6 -> 0
- removed copper zone on F.Cu, net +3V3
- removed copper zone on B.Cu, net GATE
- removed copper zone on F.Cu, net GATE
