File: hardware/kicad/opensolder.kicad_sch (KiCad schematic)
At the start: 0 parts

Commit message: Schematic update.
Other:
- sheet AC renamed DC

Commit message: lsdk
Other:
- note added: "Analogna PID kontrola"
Changed lines of the file:
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@@
 		(rev "1.1")
 		(comment 1 "Licence: GPL-3.0")
-		(comment 2 "Designer: Håvard Jakobsen")
+		(comment 2 "Designer: Nenad Tepavac")
 		(comment 4 "OpenSolder - JBC T245 compatible soldering station")
 	)
+	(text "Analogna PID kontrola"
+		(exclude_from_sim no)
+		(at 138.176 118.872 0)
+		(effects
+			(font
+				(size 6.35 6.35)
+			)
+		)
+	)
 	(sheet
